File: electrical/dreamland-biennale-electrical.sch (KiCad schematic (older format))
At the start: 8 parts

Commit message: Funciton changes to the drawings.
Parts:
- removed b-cb: Bench-control-box, symbol Bench-control-box
- removed ca-cb: Carousel-control-box, symbol Carousel-control-box
- removed lc-cb: lower-carousel-control-box, symbol lower-carousel-control-box
- removed lp-cb1, lp-cb2, lp-cb3: lamppost-control-box, symbol lamppost-control-box
- removed m-cb: Main-control-box, symbol Main-control-box
- removed sr: slip-ring, symbol slip-ring
Changed lines of the file:
@@
 $Descr A4 11693 8268
 encoding utf-8
-Sheet 1 5
-Title "Dreamland main outline"
+Sheet 1 2
+Title ""
 Date "2000-12-31"
-Rev "1b"
-Comp "Flux Foundation"
+Rev "1a"
+Comp "Flux Foudnation"
 Comment1 ""
 Comment2 ""
@@
 Comment4 ""
 $EndDescr
-$Comp
-L lamppost-control-box lp-cb1
-U 1 1 585D79F4
-P 7450 1800
-F 0 "lp-cb1" H 7850 2150 60  0000 C CNN
-F 1 "lamppost-control-box" H 7450 2600 60  0000 C CNN
-F 2 "" H 7450 1800 60  0001 C CNN
-F 3 "" H 7450 1800 60  0001 C CNN
-	1    7450 1800
-	1    0    0    -1
-$EndComp
-$Comp
-L lamppost-control-box lp-cb2
-U 1 1 585D7A36
-P 7450 2400
-F 0 "lp-cb2" H 7850 2750 60  0000 C CNN
-F 1 "lamppost-control-box" H 7450 3200 60  0000 C CNN
-F 2 "" H 7450 2400 60  0001 C CNN
-F 3 "" H 7450 2400 60  0001 C CNN
-	1    7450 2400
-	1    0    0    -1
-$EndComp
-$Comp
-L lamppost-control-box lp-cb3
-U 1 1 585D7A61
-P 7450 3000
-F 0 "lp-cb3" H 7850 3350 60  0000 C CNN
-F 1 "lamppost-control-box" H 7450 3800 60  0000 C CNN
-F 2 "" H 7450 3000 60  0001 C CNN
-F 3 "" H 7450 3000 60  0001 C CNN
-	1    7450 3000
-	1    0    0    -1
-$EndComp
-$Comp
-L Carousel-control-box ca-cb
-U 1 1 585D8647
-P 7450 4700
-F 0 "ca-cb" H 7850 5000 60  0000 C CNN
-F 1 "Carousel-control-box" H 7450 5500 60  0000 C CNN
-F 2 "" H 7450 4700 60  0001 C CNN
-F 3 "" H 7450 4700 60  0001 C CNN
-	1    7450 4700
-	1    0    0    -1
-$EndComp
-$Comp
-L Main-control-box m-cb
-U 1 1 585D8A23
-P 2750 3300
-F 0 "m-cb" H 3600 2400 60  0000 C CNN
-F 1 "Main-control-box" H 2750 4100 60  0000 C CNN
-F 2 "" H 2650 3650 60  0001 C CNN
-F 3 "" H 2650 3650 60  0001 C CNN
-	1    2750 3300
-	1    0    0    -1
-$EndComp
-$Comp
-L Bench-control-box b-cb
-U 1 1 585D8B2F
-P 7450 6000
-F 0 "b-cb" H 7850 6350 60  0000 C CNN
-F 1 "Bench-control-box" H 7450 6800 60  0000 C CNN
-F 2 "" H 7450 6000 60  0001 C CNN
-F 3 "" H 7450 6000 60  0001 C CNN
-	1    7450 6000
-	1    0    0    -1
-$EndComp
-$Comp
-L lower-carousel-control-box lc-cb
-U 1 1 585D901F
-P 7450 4150
-F 0 "lc-cb" H 7850 4500 60  0000 C CNN
-F 1 "lower-carousel-control-box" H 7450 4950 60  0000 C CNN
-F 2 "" H 7450 4150 60  0001 C CNN
-F 3 "" H 7450 4150 60  0001 C CNN
-	1    7450 4150
-	1    0    0    -1
-$EndComp
-Wire Wire Line
-	3950 4000 3950 5500
-Wire Wire Line
-	3950 5500 6700 5500
-Wire Wire Line
-	3950 3900 4100 3900
-Wire Wire Line
-	4100 3900 4100 5350
-Wire Wire Line
-	4100 5350 6700 5350
-$Comp
-L slip-ring sr
-U 1 1 585D91D1
-P 5750 4400
-F 0 "sr" H 6200 4400 60  0000 C CNN
-F 1 "slip-ring" H 5750 4900 60  0000 C CNN
-F 2 "" H 5600 4400 60  0001 C CNN
-F 3 "" H 5600 4400 60  0001 C CNN
-	1    5750 4400
-	1    0    0    -1
-$EndComp
 $Sheet
-S 6850 850  1300 1850
-U 585D935B
-F0 "lamppost_internals" 60
-F1 "lamppost.sch" 60
-$EndSheet
-Wire Wire Line
-	3950 2650 3950 1150
-Wire Wire Line
-	3950 1150 6700 1150
-Wire Wire Line
-	3950 2750 4150 2750
-Wire Wire Line
-	4150 2750 4150 1300
-Wire Wire Line
-	4150 1300 6700 1300
-Wire Wire Line
-	3950 2900 4300 2900
-Wire Wire Line
-	4300 2900 4300 1750
-Wire Wire Line
-	4300 1750 6700 1750
-Wire Wire Line
-	3950 3000 4450 3000
-Wire Wire Line
-	4450 3000 4450 1900
-Wire Wire Line
-	4450 1900 6700 1900
-Wire Wire Line
-	3950 3150 4600 3150
-Wire Wire Line
-	4600 3150 4600 2350
-Wire Wire Line
-	4600 2350 6700 2350
-Wire Wire Line
-	3950 3250 4750 3250
-Wire Wire Line
-	4750 3250 4750 2500
-Wire Wire Line
-	4750 2500 6700 2500
-Wire Wire Line
-	6450 4050 6700 4050
-Wire Wire Line
-	6450 4150 6700 4150
-Wire Wire Line
-	6450 4250 6700 4250
-Wire Wire Line
-	3950 3750 4350 3750
-Wire Wire Line
-	4350 3750 4350 4150
-Wire Wire Line
-	4350 4150 5100 4150
-Wire Wire Line
-	3950 3650 4500 3650
-Wire Wire Line
-	4500 3650 4500 4050
-Wire Wire Line
-	4500 4050 5100 4050
-Wire Wire Line
-	3950 3500 4600 3500
-Wire Wire Line
-	4600 3500 4600 3650
-Wire Wire Line
-	4600 3650 6700 3650
-Wire Wire Line
-	3950 3400 4700 3400
-Wire Wire Line
-	4700 3400 4700 3500
-Wire Wire Line
-	4700 3500 6700 3500
-$Sheet
-S 6750 3200 1450 1350
-U 585D9C03
-F0 "carousel_internals" 60
-F1 "carousel.sch" 60
-$EndSheet
-$Sheet
-S 6850 5100 1250 650
-U 585D9C30
-F0 "bench_internals" 60
-F1 "bench.sch" 60
-$EndSheet
-$Sheet
-S 1700 2250 2150 2050
-U 585D9EED
+S 1400 1800 2400 2500
+U 585FE4A1
 F0 "main_control_box_internals" 60
 F1 "main_control_box_internals.sch" 60
-$EndSheet
-$Sheet
-S 1700 5000 1150 550
-U 585D9FF9
-F0 "network_layout" 60
-F1 "network_layout.sch" 60
+F2 "Power_in" I L 1400 2150 60
+F3 "Data_in" I L 1400 3600 60
+F4 "Lamppost_1_pwr" I R 3800 2050 60
+F5 "Lamppost_2_pwr" I R 3800 2200 60
+F6 "Lamppost_3_pwr" I R 3800 2350 60
+F7 "Carousel_bottom_pwr" I R 3800 2500 60
+F8 "Carousel_top_pwr" I R 3800 2650 60
+F9 "Benches_pwr" I R 3800 2800 60
+F10 "Lamppost_1_data" I R 3800 3150 60
+F11 "Lamppost_2_data" I R 3800 3300 60
+F12 "Lamppost_3_data" I R 3800 3450 60
+F13 "Carousel_bottom_data" I R 3800 3600 60
+F14 "Catousel_top_data" I R 3800 3750 60
+F15 "Benches_data" I R 3800 3900 60
 $EndSheet
 $EndSCHEMATC

Commit message: Initial revision of the main control box.
Parts:
- added sr?: slip-ring, symbol slip-ring
Changed lines of the file:
@@
 encoding utf-8
 Sheet 1 2
-Title ""
+Title "Dreamland Overview"
 Date "2000-12-31"
 Rev "1a"
@@
 $EndDescr
 $Sheet
-S 1400 1800 2400 2500
+S 1400 1900 2400 2500
 U 585FE4A1
 F0 "main_control_box_internals" 60
 F1 "main_control_box_internals.sch" 60
-F2 "Power_in" I L 1400 2150 60
-F3 "Data_in" I L 1400 3600 60
-F4 "Lamppost_1_pwr" I R 3800 2050 60
-F5 "Lamppost_2_pwr" I R 3800 2200 60
-F6 "Lamppost_3_pwr" I R 3800 2350 60
-F7 "Carousel_bottom_pwr" I R 3800 2500 60
-F8 "Carousel_top_pwr" I R 3800 2650 60
-F9 "Benches_pwr" I R 3800 2800 60
-F10 "Lamppost_1_data" I R 3800 3150 60
-F11 "Lamppost_2_data" I R 3800 3300 60
-F12 "Lamppost_3_data" I R 3800 3450 60
-F13 "Carousel_bottom_data" I R 3800 3600 60
-F14 "Catousel_top_data" I R 3800 3750 60
-F15 "Benches_data" I R 3800 3900 60
+F2 "Power_in" I L 1400 2250 60
+F3 "Data_in" I L 1400 3700 60
+F4 "Lamppost_1_pwr" I R 3800 2100 60
+F5 "Lamppost_2_pwr" I R 3800 2400 60
+F6 "Lamppost_3_pwr" I R 3800 2700 60
+F7 "Carousel_bottom_pwr" I R 3800 3300 60
+F8 "Carousel_top_pwr" I R 3800 3600 60
+F9 "Benches_pwr" I R 3800 3000 60
+F10 "Lamppost_1_data" I R 3800 2200 60
+F11 "Lamppost_2_data" I R 3800 2500 60
+F12 "Lamppost_3_data" I R 3800 2800 60
+F13 "Carousel_bottom_data" I R 3800 3400 60
+F14 "Catousel_top_data" I R 3800 3700 60
+F15 "Benches_data" I R 3800 3100 60
+F16 "Access_point" I L 1400 3900 60
 $EndSheet
+$Comp
+L slip-ring sr?
+U 1 1 5864171C
+P 6050 4050
+F 0 "sr?" H 6500 4050 60  0000 C CNN
+F 1 "slip-ring" H 6050 4550 60  0000 C CNN
+F 2 "" H 5900 4050 60  0001 C CNN
+F 3 "" H 5900 4050 60  0001 C CNN
+	1    6050 4050
+	1    0    0    -1
+$EndComp
 $EndSCHEMATC

Commit message: Finished dreamland overview.
Parts:
- removed sr?: slip-ring, symbol slip-ring
- added sr?: slip-ring, symbol slip-ring
Other:
- note added: "All three lamposts use the same \ncontrol box architecture."
- note added: "Notes:\n1) All pwr is 230V @ 50Hz\n2) All pwr conductors are romex 14-3\n3) All data lines are Cat-5e"
Changed lines of the file:
@@
 $Descr A4 11693 8268
 encoding utf-8
-Sheet 1 2
+Sheet 1 6
 Title "Dreamland Overview"
-Date "2000-12-31"
-Rev "1a"
+Date "2016-12-28"
+Rev "1b"
 Comp "Flux Foudnation"
 Comment1 ""
@@
 F16 "Access_point" I L 1400 3900 60
 $EndSheet
+$Sheet
+S 4900 800  2000 1350
+U 58643230
+F0 "lamppost_control_box" 60
+F1 "lampost_internals.sch" 60
+F2 "Lamppost_data" I L 4900 1600 60
+F3 "Lamppost_power" I L 4900 1000 60
+F4 "light_1" I R 6900 950 60
+F5 "light_2" I R 6900 1050 60
+F6 "light_3" I R 6900 1150 60
+F7 "light_4" I R 6900 1250 60
+F8 "light_5" I R 6900 1350 60
+F9 "light_6" I R 6900 1450 60
+F10 "light_7" I R 6900 1550 60
+F11 "button_switch" I R 6900 1700 60
+F12 "button_light" I R 6900 1800 60
+F13 "poofer" I R 6900 1950 60
+$EndSheet
+Wire Bus Line
+	3800 2100 4100 2100
+Wire Bus Line
+	4100 2100 4100 1000
+Wire Bus Line
+	4100 1000 4900 1000
+Wire Bus Line
+	3800 2200 4200 2200
+Wire Bus Line
+	4200 2200 4200 1600
+Wire Bus Line
+	4200 1600 4900 1600
+Text Notes 4000 2600 0    60   ~ 0
+All three lamposts use the same \ncontrol box architecture.
+Wire Bus Line
+	3800 2400 3900 2400
+Wire Bus Line
+	3800 2500 3900 2500
+Wire Bus Line
+	3800 2700 3900 2700
+Wire Bus Line
+	3800 2800 3900 2800
+Wire Notes Line
+	3950 2000 3950 2850
+Wire Notes Line
+	3850 2000 3950 2000
+Wire Notes Line
+	3850 2000 3850 2850
+Wire Notes Line
+	3850 2850 3950 2850
+Text GLabel 7200 950  2    60   Input ~ 0
+light_bar
+Wire Bus Line
+	6900 950  7200 950
+Text GLabel 7200 1750 2    60   Input ~ 0
+LED_Button
+Wire Bus Line
+	6900 1700 7200 1700
+Wire Bus Line
+	7200 1700 7200 1800
+Wire Bus Line
+	7200 1800 6900 1800
+Text GLabel 7200 1950 2    60   Input ~ 0
+12V_solenoid
+Wire Bus Line
+	6900 1950 7200 1950
+$Sheet
+S 4898 2902 1902 298
+U 5864B548
+F0 "benches_internals" 60
+F1 "benches_control_box.sch" 60
+F2 "benches_pwr" I L 4898 3000 60
+F3 "benches_data" I L 4898 3100 60
+F4 "benches_light_string" I R 6800 3050 60
+$EndSheet
+Wire Bus Line
+	3800 3100 4900 3100
+Wire Bus Line
+	4900 3000 3800 3000
+Text GLabel 7000 3050 1    60   Input ~ 0
+inner_bench_1
+Text GLabel 7200 3050 1    60   Input ~ 0
+inner_bench_2
+Text GLabel 7400 3050 1    60   Input ~ 0
+inner_bench_3
+Text GLabel 7600 3050 1    60   Input ~ 0
+outer_bench_1
+Text GLabel 7800 3050 1    60   Input ~ 0
+outer_bench_2
+Text GLabel 8000 3050 1    60   Input ~ 0
+outer_bench_3
+Text GLabel 8200 3050 1    60   Input ~ 0
+kaleidoscope_1
+Text GLabel 8400 3050 1    60   Input ~ 0
+kaleidoscope_2
+Text GLabel 8600 3050 1    60   Input ~ 0
+kaleidoscope_3
+Wire Bus Line
+	6800 3050 8600 3050
+$Sheet
+S 4900 3500 2000 1050
+U 5864D7E5
+F0 "carousel_bottom_internals" 60
+F1 "carousel_bottom_control_box.sch" 60
+F2 "carousel_bottom_pwr" I L 4900 3600 60
+F3 "led_1" I R 6900 3600 60
+F4 "led_2" I R 6900 3700 60
+F5 "led_3" I R 6900 3800 60
+F6 "led_4" I R 6900 3900 60
+F7 "led_5" I R 6900 4000 60
+F8 "led_6" I R 6900 4100 60
+F9 "led_7" I R 6900 4200 60
+F10 "led_8" I R 6900 4300 60
+F11 "led_9" I R 6900 4400 60
+F12 "carousel_bottom_data" I L 4900 3700 60
+$EndSheet
+Text GLabel 7300 3600 2    60   Input ~ 0
+carousel_lower_led_bar
+Wire Bus Line
+	6900 3600 7300 3600
+Wire Bus Line
+	4900 3600 4750 3600
+Wire Bus Line
+	4750 3600 4750 3300
+Wire Bus Line
+	4750 3300 3800 3300
+Wire Bus Line
+	3800 3400 4650 3400
+Wire Bus Line
+	4650 3400 4650 3700
+Wire Bus Line
+	4650 3700 4900 3700
+Wire Bus Line
+	3800 3700 3900 3700
+Wire Bus Line
+	3900 3700 3900 4700
+Wire Bus Line
+	3900 4700 1000 4700
+Wire Bus Line
+	3800 3600 4000 3600
+Wire Bus Line
+	4000 3600 4000 4800
+Wire Bus Line
+	4000 4800 1100 4800
+Wire Bus Line
+	1100 4800 1100 5100
 $Comp
 L slip-ring sr?
-U 1 1 5864171C
-P 6050 4050
-F 0 "sr?" H 6500 4050 60  0000 C CNN
-F 1 "slip-ring" H 6050 4550 60  0000 C CNN
-F 2 "" H 5900 4050 60  0001 C CNN
-F 3 "" H 5900 4050 60  0001 C CNN
-	1    6050 4050
+U 1 1 5864F4FF
+P 2100 5450
+F 0 "sr?" H 2550 5450 60  0000 C CNN
+F 1 "slip-ring" H 2100 5950 60  0000 C CNN
+F 2 "" H 1950 5450 60  0001 C CNN
+F 3 "" H 1950 5450 60  0001 C CNN
+	1    2100 5450
 	1    0    0    -1
 $EndComp
+Wire Bus Line
+	1450 5200 1000 5200
+Wire Bus Line
+	1000 5200 1000 4700
+Wire Bus Line
+	1100 5100 1450 5100
+$Sheet
+S 3700 5000 1600 1500
+U 5865044B
+F0 "carousel_top_control_box" 60
+F1 "carousel_top_internals.sch" 60
+F2 "carousel_top_pwr" I L 3700 5100 60
+F3 "carousel_top_data" I L 3700 5200 60
+F4 "rotary_encoder" I L 3700 5300 60
+F5 "led_1" I R 5300 5100 60
+F6 "led_2" I R 5300 5200 60
+F7 "led_3" I R 5300 5300 60
+F8 "led_4" I R 5300 5400 60
+F9 "led_5" I R 5300 5500 60
+F10 "led_6" I R 5300 5600 60
+F11 "led_7" I R 5300 5700 60
+F12 "led_8" I R 5300 5800 60
+F13 "led_9" I R 5300 5900 60
+F14 "poofer_1" I R 5300 6100 60
+F15 "poofer_2" I R 5300 6200 60
+F16 "poofer_3" I R 5300 6300 60
+F17 "poofer_4" I R 5300 6400 60
+$EndSheet
+Wire Bus Line
+	2800 5100 3700 5100
+Wire Bus Line
+	2800 5200 3700 5200
+Wire Bus Line
+	3700 5300 2800 5300
+Text GLabel 5600 5100 2    60   Input ~ 0
+light_bar
+Text GLabel 5600 6100 2    60   Input ~ 0
+12V_solenoid
+Wire Bus Line
+	5300 5100 5600 5100
+Wire Bus Line
+	5300 6100 5600 6100
+Text Notes 900  7550 0    60   ~ 0
+Notes:\n1) All pwr is 230V @ 50Hz\n2) All pwr conductors are romex 14-3\n3) All data lines are Cat-5e
 $EndSCHEMATC
